File: roxie-lcd.sch (KiCad schematic (older format))
At the start: 25 parts, among them J1 JTAG, J2 LCD_SPI, J3 VESC, U1 AMS1117-3.3, U2 STM32F103C8T6, Y1 8MHz

Commit message: Change connectors
Parts:
- removed FB1: Ferrite_Bead_Small, Inductor_SMD:L_0805_2012Metric, symbol Device:Ferrite_Bead_Small
- added C1: 100n, Capacitor_SMD:C_0402_1005Metric, symbol Device:C
- added C14, C15, C16: 100n, Capacitor_SMD:C_0402_1005Metric, symbol Device:C_Small
- added C4: 22u, Capacitor_SMD:C_0805_2012Metric, symbol Device:C
- added J4: UP, Connector_PinHeader_2.54mm:PinHeader_1x02_P2.54mm_Vertical, symbol Switch:SW_SPST
- added J5: DOWN, Connector_PinHeader_2.54mm:PinHeader_1x02_P2.54mm_Vertical, symbol Switch:SW_SPST
- added J6: SELECT, Connector_PinHeader_2.54mm:PinHeader_1x02_P2.54mm_Vertical, symbol Switch:SW_SPST
- added R3, R4, R5, R6: 10k, Resistor_SMD:R_0603_1608Metric, symbol Device:R_Small
- C11: renamed from C9; footprint Capacitor_SMD:C_0402_1005Metric -> Capacitor_SMD:C_0603_1608Metric
- C12: renamed from C10; value 20p -> 15p
- C13: renamed from C11; value 20p -> 15p
- C3: renamed from C2; value 10u -> 22u
- J1: footprint Connector_JST:JST_PH_B4B-PH-K_1x04_P2.00mm_Vertical -> Connector_PinHeader_2.54mm:PinHeader_1x04_P2.54mm_Horizontal
- J2: footprint Connector_JST:JST_PH_B11B-PH-K_1x11_P2.00mm_Vertical -> Connector_PinHeader_2.54mm:PinHeader_1x11_P2.54mm_Vertical
- J3: footprint Connector_JST:JST_PH_B4B-PH-K_1x04_P2.00mm_Vertical -> Connector_JST:JST_PH_S4B-PH-K_1x04_P2.00mm_Horizontal
- renumbered C8 to C10, C1 to C2, C3 to C5, C4 to C6, C5 to C7, C6 to C8, C7 to C9, R3 to R7, R4 to R8
Connections:
- net labels added: BTN_DOWN, BTN_SELECT, BTN_UP, CAN_RX
- net labels removed: CANRX, NRST
- wire segments 94 -> 131
- no-connect marks 27 -> 24
Other:
- note added: "AN2586 section 1.2\n"
- note added: "CL = CL1 x CL2 / (CL1 + CL2) + Cstray where: Cstray is the pin capacitance \nand board or trace PCB-related capacitance. \nTypically, it is between 2 pF and 7 pF. Maximum value of CL1 and CL2 is 15 pF"
- moved on the sheet: C10, C11, C12, C13, C2, C3, C5, C6, C7, C8, C9, D1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
